File: Schematics/ir_shield/ir_shield.sch (KiCad schematic (older format))
At the start: 51 parts, among them Q1 Q_Photo_NPN, Q2 Q_Photo_NPN, Q3 Q_Photo_NPN, Q4 Q_Photo_NPN, Q5 Q_NMOS, U1 LM6132

Commit message: added some changes
Parts:
- R10, R11: value 100R -> 2k
- RV3, RV4: value 100k -> 20k
