File: Schematics/misc_shield/misc_shield.kicad_pcb (KiCad board)
At the start: 4 copper layers, 68.6 x 53.3 mm, 30 parts, among them J1 Conn_1x1_Female, J10 Conn_1x1_Female, J11 Conn_1x1_Female, J12 Conn_1x1_Female, J2 Conn_1x1_Female, J3 Conn_1x1_Female, J4 Conn_1x1_Female, J5 Conn_1x1_Female, J6 Conn_1x1_Female, J7 Conn_1x1_Female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

Commit message: added some changes
Parts:
- added J13: Conn_1x1_Female, ECE3400:PinSocket_1x1, F.Cu at (172.7, 114.3)
- added J14: Conn_1x1_Female, ECE3400:PinSocket_1x1, F.Cu at (172.7, 111.8)
- added J15: Conn_1x1_Female, ECE3400:PinSocket_1x1, F.Cu at (172.7, 116.8)
- added JP8: Jumper, ECE3400:Jumper, F.Cu at (172.7, 124.5)
- added R6: 1k, ECE3400:Resistor_THT, B.Cu at (172.7, 119.4)
Routing:
- net GND: track 104.8 -> 109.8 mm
- net +5V: track 63.5 -> 68.6 mm
- net Net-(JP8-Pad2): track 0.00 -> 2.54 mm
- net /ANALOG_C: track 0.00 -> 2.54 mm
Other:
- board text removed: "misc_shield.kicad_pcb"
