File: Schematics/misc_shield/misc_shield.sch (KiCad schematic (older format))
At the start: 30 parts, among them J1 Conn_1x1_Female, J10 Conn_1x1_Female, J11 Conn_1x1_Female, J12 Conn_1x1_Female, J2 Conn_1x1_Female, J3 Conn_1x1_Female, J4 Conn_1x1_Female, J5 Conn_1x1_Female, J6 Conn_1x1_Female, J7 Conn_1x1_Female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

Commit message: added some changes
Parts:
- added J13, J14, J15: Conn_1x1_Female, ECE3400:PinSocket_1x1, symbol ECE3400:Conn_1x1_Female
- added JP8: Jumper, ECE3400:Jumper, symbol ECE3400:Jumper
- added R6: 1k, ECE3400:Resistor_THT, symbol ECE3400:R
Connections:
- net +5V: now also J13.1 (Pin_1)
- net GND: now also J15.1 (Pin_1)
- net at A1.13 (A4/SDA): now also JP8.1
- new net: JP8.2, R6.1
- new net ANALOG_C: J14.1 (Pin_1), R6.2
- no-connect marks 20 -> 19
Other:
- moved on the sheet: J1, J10, J11, J12, J2, J3, J4, J5, J6, J7, J8, J9
