File: Schematics/sound_shield/sound_shield.kicad_pcb (KiCad board)
At the start: 4 copper layers, 68.6 x 53.3 mm, 25 parts, among them U1 LM6132

Commit message: added some changes
Other:
- board text removed: "misc_shield.kicad_pcb"
Changed lines of the file:
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@@
   (general
     (thickness 1.6)
-    (drawings 29)
+    (drawings 28)
     (tracks 169)
     (zones 0)
@@
     (at 142.24 95.5825 270)
     (attr smd)
-    (fp_text reference C2 (at 2.2075 0) (layer F.SilkS)
+    (fp_text reference C2 (at -2.8725 0) (layer F.SilkS)
       (effects (font (size 1 1) (thickness 0.15)))
     )
@@
     (at 167.64 100.6625 270)
     (attr smd)
-    (fp_text reference C3 (at 2.2075 0) (layer F.SilkS)
+    (fp_text reference C3 (at -2.8725 0) (layer F.SilkS)
       (effects (font (size 1 1) (thickness 0.15)))
     )
@@
     )
   )
-  (gr_text misc_shield.kicad_pcb (at 194.31 186.055) (layer Dwgs.User)
-    (effects (font (size 1.27 1.27) (thickness 0.127)))
-  )
   (gr_text - (at 269.875 193.04) (layer Dwgs.User)
     (effects (font (size 1.27 1.27) (thickness 0.127)))
@@
   (gr_line (start 139.7 132.08) (end 139.7 127) (layer Edge.Cuts) (width 0.2))
   (gr_line (start 129.54 83.82) (end 177.8 83.82) (layer Edge.Cuts) (width 0.2))
-  (gr_line (start 111.76 132.08) (end 114.3 132.08) (layer Edge.Cuts) (width 0.15))
-  (gr_line (start 111.76 78.74) (end 111.76 132.08) (layer Edge.Cuts) (width 0.15))
-  (gr_line (start 127 78.74) (end 111.76 78.74) (layer Edge.Cuts) (width 0.15))
-  (gr_line (start 127 81.28) (end 127 78.74) (layer Edge.Cuts) (width 0.15))
-  (gr_line (start 129.54 81.28) (end 127 81.28) (layer Edge.Cuts) (width 0.15))
-  (gr_line (start 129.54 83.82) (end 129.54 81.28) (layer Edge.Cuts) (width 0.15))
-  (gr_line (start 177.8 91.44) (end 177.8 83.82) (layer Edge.Cuts) (width 0.15))
-  (gr_line (start 180.34 91.44) (end 177.8 91.44) (layer Edge.Cuts) (width 0.15))
-  (gr_line (start 180.34 96.52) (end 180.34 91.44) (layer Edge.Cuts) (width 0.15))
-  (gr_line (start 180.34 96.52) (end 177.8 96.52) (layer Edge.Cuts) (width 0.15))
-  (gr_line (start 180.34 124.46) (end 180.34 96.52) (layer Edge.Cuts) (width 0.15))
-  (gr_line (start 177.8 124.46) (end 180.34 124.46) (layer Edge.Cuts) (width 0.15))
-  (gr_line (start 177.8 124.46) (end 177.8 127) (layer Edge.Cuts) (width 0.15))
+  (gr_line (start 111.76 132.08) (end 114.3 132.08) (layer Edge.Cuts) (width 0.2))
+  (gr_line (start 111.76 78.74) (end 111.76 132.08) (layer Edge.Cuts) (width 0.2))
+  (gr_line (start 127 78.74) (end 111.76 78.74) (layer Edge.Cuts) (width 0.2))
+  (gr_line (start 127 81.28) (end 127 78.74) (layer Edge.Cuts) (width 0.2))
+  (gr_line (start 129.54 81.28) (end 127 81.28) (layer Edge.Cuts) (width 0.2))
+  (gr_line (start 129.54 83.82) (end 129.54 81.28) (layer Edge.Cuts) (width 0.2))
+  (gr_line (start 177.8 91.44) (end 177.8 83.82) (layer Edge.Cuts) (width 0.2))
+  (gr_line (start 180.34 91.44) (end 177.8 91.44) (layer Edge.Cuts) (width 0.2))
+  (gr_line (start 180.34 96.52) (end 180.34 91.44) (layer Edge.Cuts) (width 0.2))
+  (gr_line (start 180.34 96.52) (end 177.8 96.52) (layer Edge.Cuts) (width 0.2))
+  (gr_line (start 180.34 124.46) (end 180.34 96.52) (layer Edge.Cuts) (width 0.2))
+  (gr_line (start 177.8 124.46) (end 180.34 124.46) (layer Edge.Cuts) (width 0.2))
+  (gr_line (start 177.8 124.46) (end 177.8 127) (layer Edge.Cuts) (width 0.2))
   (gr_line (start 177.8 127) (end 177.8 124.46) (layer Edge.Cuts) (width 0.15))
   (gr_line (start 137.16 132.08) (end 139.7 132.08) (layer Edge.Cuts) (width 0.2))
@@
   (segment (start 124.46 88.9) (end 124.46 91.44) (width 0.25) (layer B.Solder) (net 32))
   (segment (start 132.08 93.98) (end 134.62 93.98) (width 0.25) (layer B.Solder) (net 32))
+  (segment (start 121.92 86.36) (end 124.46 86.36) (width 0.25) (layer B.Solder) (net 32))
+  (segment (start 124.46 88.9) (end 124.46 86.36) (width 0.25) (layer B.Solder) (net 32))
   (segment (start 160.02 99.06) (end 160.02 96.52) (width 0.25) (layer B.Solder) (net 33))
   (segment (start 160.02 96.52) (end 160.02 93.98) (width 0.25) (layer B.Solder) (net 33))
@@
   (segment (start 144.78 99.06) (end 147.32 99.06) (width 0.25) (layer B.Solder) (net 37))
   (segment (start 147.32 96.52) (end 147.32 91.44) (width 0.25) (layer B.Solder) (net 37))
-  (segment (start 121.92 86.36) (end 124.46 86.36) (width 0.25) (layer B.Solder) (net 32))
-  (segment (start 124.46 88.9) (end 124.46 86.36) (width 0.25) (layer B.Solder) (net 32))
   (segment (start 147.32 129.54) (end 147.32 125.73) (width 0.25) (layer B.Solder) (net 38))
   (segment (start 147.32 124.46) (end 147.32 125.73) (width 0.25) (layer B.Solder) (net 38))
